File: PCB files/Metal Detector.sch (EAGLE design)
At the start: 52 parts, among them IC1 NE5534AD, IC2 ESP32-WROOM-32UE-N4, IC3 CP2102, Q1 IRF740, Q2 BC556, Q3 MBT3904DW1T1, T1 BC547, X1 A1944-50

Commit message: Add files via upload
Deleted sheet 2 and include content to sheet 1 for software limitations after that edited sheet 1
Parts:
- removed C10, C15, C6: 100nF/ 50v, rcl:C-EUC0603
- removed C11: 4u7F/16v, rcl:C-EUC0603
- removed C12, C9: 1nF / 50 V, rcl:C-EUC0603
- removed C13: 100uF/ 6.3V, rcl:C-EUC0603
- removed C14: 1uF/ 16v, rcl:C-EUC0603
- removed C16, C8: 1uF/16v, rcl:C-EUC0603
- removed D5, D6, D7: ESD05V88D-LC, ESD05V88D-LC:ESD05V88D-LC
- removed F1: 500mA, SparkFun-PowerIC:PTCSMD
- removed IC2: ESP32-WROOM-32UE-N4, ESP32-WROOM-32UE-N4:ESP32-WROOM-32UE-N4
- removed IC3: CP2102, CP2102:CP2102
- removed JP1: (no value), SparkFun-Connectors:USB_MICROB_PLUGCONN-11752
- removed Q3: MBT3904DW1T1, esp32-thing-temp:MBT3904DW1T1
- removed R11, R13, R14, R15, R16: 10K, rcl:R-EU_R0603
- removed R12: 4K7, rcl:R-EU_R0603
- removed S1: RESET, SparkFun-Electromechanical:SWITCH-MOMENTARY-2SMD-4.6X2.8MM
- removed S2: BTN-0, SparkFun-Electromechanical:SWITCH-MOMENTARY-2SMD-4.6X2.8MM
- added C17, C18: 1nF / 50 V, rcl:C-EUC0603
- added C19: 100uF/ 6.3V, rcl:C-EUC0603
- added C20: 1uF/ 16v, rcl:C-EUC0603
- added C21, C23, C25: 100nF/ 50v, rcl:C-EUC0603
- added C22, C26: 1uF/16v, rcl:C-EUC0603
- added C24: 4u7F/16v, rcl:C-EUC0603
- added D4, D8, D9: ESD05V88D-LC, ESD05V88D-LC:ESD05V88D-LC
- added F2: 500mA, SparkFun-PowerIC:PTCSMD
- added FRAME3: FRAME-LEDGER, SparkFun-Aesthetics:FRAME-LEDGER
- added IC4: ESP32-WROOM-32UE-N4, ESP32-WROOM-32UE-N4:ESP32-WROOM-32UE-N4
- added IC5: CP2102, CP2102:CP2102
- added JP2: (no value), SparkFun-Connectors:USB_MICROB_PLUGCONN-11752
- added Q4: MBT3904DW1T1, esp32-thing-temp:MBT3904DW1T1
- added R17, R18, R20, R21, R22: 10K, rcl:R-EU_R0603
- added R19: 4K7, rcl:R-EU_R0603
- added S3: RESET, SparkFun-Electromechanical:SWITCH-MOMENTARY-2SMD-4.6X2.8MM
- added S4: BTN-0, SparkFun-Electromechanical:SWITCH-MOMENTARY-2SMD-4.6X2.8MM
Connections:
- removed net N$14: Q3Q1.B, R14.2
- removed net N$15: Q3Q2.B, R15.2
- removed net N$16: IC3.TXD, R16.1
- new net N$18: Q4Q2.B, R21.2
- new net N$19: IC5.TXD, R22.1
- new net VCC_USB: D9.1, F2.1, JP2.VCC
- net 3V3: now also C19.2, C20.2, IC4.3V3; no longer C13.2, C14.2, IC2.3V3
- net ACTıVE: now also IC5.!SUSPEND; no longer IC3.!SUSPEND
- net CLK: now also IC4.NC_4; no longer IC2.NC_4
- net CMD: now also IC4.NC_3; no longer IC2.NC_3
- net DCD: now also IC5.DCD; no longer IC3.DCD
- net DSR: now also IC5.DSR; no longer IC3.DSR
- net DTR: now also IC5.DTR, Q4Q2.E, R20.1; no longer IC3.DTR, Q3Q2.E, R14.1
- net EN: now also C18.1, IC4.EN, Q4Q1.C, R18.1, S3.2; no longer C12.1, IC2.EN, Q3Q1.C, R13.1, S1.2
- net GND: now also C17.2, C18.2, C19.1, C20.1, C21.1, C22.1, C23.1, C24.1, C25.1, C26.1, D4.2, D8.2, D9.2, IC4.GND_1, IC4.GND_10, IC4.GND_11, IC4.GND_12, IC4.GND_2, IC4.GND_3, IC4.GND_4, IC4.GND_5, IC4.GND_6, IC4.GND_7, IC4.GND_8, IC4.GND_9, IC5.GND, JP2.GND, R19.1, S3.1, S4.1; no longer C10.1, C11.1, C12.2, C13.1, C14.1, C15.1, C16.1, C6.1, C8.1, C9.2, D5.2, D6.2, D7.2, IC2.GND_1, IC2.GND_10, IC2.GND_11, IC2.GND_12, IC2.GND_2, IC2.GND_3, IC2.GND_4, IC2.GND_5, IC2.GND_6, IC2.GND_7, IC2.GND_8, IC2.GND_9, IC3.GND, JP1.GND, R12.1, S1.1, S2.1
- net IO0: now also C17.1, IC4.IO0, Q4Q2.C, R17.1, S4.2; no longer C9.1, IC2.IO0, Q3Q2.C, R11.1, S2.2
- net IO12: now also IC4.IO12; no longer IC2.IO12
- net IO13: now also IC4.IO13, IC5.RTS; no longer IC2.IO13, IC3.RTS
- net IO14: now also IC4.IO14; no longer IC2.IO14
- net IO15: now also IC4.IO15, IC5.CTS; no longer IC2.IO15, IC3.CTS
- net IO16: now also IC4.IO16; no longer IC2.IO16
- net IO17: now also IC4.IO17; no longer IC2.IO17
- net IO18: now also IC4.IO18; no longer IC2.IO18
- net IO19: now also IC4.IO19; no longer IC2.IO19
- net IO2: now also IC4.IO2, R19.2; no longer IC2.IO2, R12.2
- net IO21: now also IC4.IO21; no longer IC2.IO21
- net IO22: now also IC4.IO22; no longer IC2.IO22
- net IO23: now also IC4.IO23, IC4.NC_7; no longer IC2.IO23, IC2.NC_7
- net IO25: now also IC4.IO25; no longer IC2.IO25
- net IO26: now also IC4.IO26; no longer IC2.IO26
- net IO27: now also IC4.IO27; no longer IC2.IO27
- net IO32: now also IC4.IO32; no longer IC2.IO32
- net IO33: now also IC4.IO33; no longer IC2.IO33
- net IO34: now also IC4.IO34; no longer IC2.IO34
- net IO35: now also IC4.IO35; no longer IC2.IO35
- net IO4: now also IC4.IO4; no longer IC2.IO4
- net IO5: now also IC4.IO5; no longer IC2.IO5
- net N$17: now also Q4Q1.B, R20.2; no longer F1.1, JP1.VCC
- net REGIN: now also C23.2, C24.2, IC5.REGIN; no longer C10.2, C11.2, IC3.REGIN
- net RI: now also IC5.RI; no longer IC3.RI
- net RTS: now also Q4Q1.E, R21.1; no longer Q3Q1.E, R15.1
- net RXD0: now also IC4.RXD0, R22.2; no longer IC2.RXD0, R16.2
- net SD0: now also IC4.NC_5; no longer IC2.NC_5
- net SD1: now also IC4.NC_6; no longer IC2.NC_6
- net SD2: now also IC4.NC_1; no longer IC2.NC_1
- net SD3: now also IC4.NC_2; no longer IC2.NC_2
- net SENSOR_VN: now also IC4.SENSOR_VN; no longer IC2.SENSOR_VN
- net SENSOR_VP: now also IC4.SENSOR_VP; no longer IC2.SENSOR_VP
- net TXD0: now also IC4.TXD0, IC5.RXD; no longer IC2.TXD0, IC3.RXD
- net USB_DN: now also D4.1, IC5.D-, JP2.D-; no longer D5.1, IC3.D-, JP1.D-
- net USB_DP: now also D8.1, IC5.D+, JP2.D+; no longer D6.1, IC3.D+, JP1.D+
- net VBUS_CP: now also C25.2, C26.2, IC5.VBUS; no longer C15.2, C16.2, IC3.VBUS
- net VCC: now also F2.2, R17.2, R18.2; no longer D7.1, F1.2, R11.2, R13.2
- net VDD_CP: now also C21.2, C22.2, IC5.VDD; no longer C6.2, C8.2, IC3.VDD
Other:
- note added: "BATTERY CHARGE &POWER REGULATORS"
- note added: "SIGNAL PROCESSING CIRCUIT"
- note removed: "Signal Processing Circuit"

Commit message: Add files via upload
Added Battery charging & power regulator and User Interface components, created board file.
Design process still on progress.
Parts:
- added DS1: NHD-12864WG-BTGH-T#N, NHD-12864WG-BTGH-T#N:NHD-12864WG-BTGH-T#N
- added IC2: BQ24133RGYR, BQ24133RGYR:BQ24133RGYR
- added IC3: MC33269D-5.0G, MC33269D-5.0G:MC33269D-5.0G
- added IC6: NCP1117DT12G, NCP1117DT12G:NCP1117DT12G
- added LS1: MCKPT-G1340-3917, MCKPT-G1340-3917:MCKPT-G1340-3917
- added R11, R12: PC16S, piher:PC16S
- added X2: DC21MMX, powersupply:DC21MMX
Changed lines of the file:
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@@
 <part name="GND20" library="SparkFun-Aesthetics" deviceset="GND" device=""/>
 <part name="GND21" library="SparkFun-Aesthetics" deviceset="GND" device=""/>
+<part name="IC2" library="BQ24133RGYR" deviceset="BQ24133RGYR" device=""/>
+<part name="X2" library="powersupply" deviceset="DC21MM" device="X"/>
+<part name="IC3" library="MC33269D-5.0G" deviceset="MC33269D-5.0G" device=""/>
+<part name="IC6" library="NCP1117DT12G" deviceset="NCP1117DT12G" device=""/>
+<part name="DS1" library="NHD-12864WG-BTGH-T#N" deviceset="NHD-12864WG-BTGH-T#N" device=""/>
+<part name="R11" library="piher" library_urn="urn:adsk.eagle:library:324" deviceset="PC16S" device="" package3d_urn="urn:adsk.eagle:package:22243/1"/>
+<part name="R12" library="piher" library_urn="urn:adsk.eagle:library:324" deviceset="PC16S" device="" package3d_urn="urn:adsk.eagle:package:22243/1"/>
+<part name="LS1" library="MCKPT-G1340-3917" deviceset="MCKPT-G1340-3917" device=""/>
 </parts>
 <sheets>
@@
 <attribute name="VALUE" x="162.56" y="474.98" size="1.778" layer="96"/>
 </instance>
+<instance part="IC2" gate="G$1" x="63.5" y="327.66" smashed="yes">
+<attribute name="NAME" x="100.33" y="347.98" size="1.778" layer="95" align="center-left"/>
+<attribute name="VALUE" x="100.33" y="345.44" size="1.778" layer="96" align="center-left"/>
+</instance>
+<instance part="X2" gate="G$1" x="27.94" y="350.52" smashed="yes"/>
+<instance part="IC3" gate="G$1" x="139.7" y="335.28" smashed="yes">
+<attribute name="NAME" x="171.45" y="342.9" size="1.778" layer="95" align="center-left"/>
+<attribute name="VALUE" x="171.45" y="340.36" size="1.778" layer="96" align="center-left"/>
+</instance>
+<instance part="IC6" gate="G$1" x="142.24" y="299.72" smashed="yes">
+<attribute name="NAME" x="173.99" y="307.34" size="1.778" layer="95" align="center-left"/>
+<attribute name="VALUE" x="173.99" y="304.8" size="1.778" layer="96" align="center-left"/>
+</instance>
+<instance part="DS1" gate="G$1" x="327.66" y="358.14" smashed="yes" rot="R90">
+<attribute name="NAME" x="354.33" y="386.08" size="1.778" layer="95" align="center-left"/>
+<attribute name="VALUE" x="354.33" y="383.54" size="1.778" layer="96" align="center-left"/>
+</instance>
+<instance part="R11" gate="G$1" x="337.82" y="335.28" smashed="yes">
+<attribute name="NAME" x="333.756" y="338.836" size="1.778" layer="95"/>
+<attribute name="VALUE" x="335.534" y="336.55" size="1.778" layer="96"/>
+</instance>
+<instance part="R12" gate="G$1" x="365.76" y="335.28" smashed="yes">
+<attribute name="NAME" x="361.696" y="338.836" size="1.778" layer="95"/>
+<attribute name="VALUE" x="363.474" y="336.55" size="1.778" layer="96"/>
+</instance>
+<instance part="LS1" gate="G$1" x="297.18" y="342.9" smashed="yes">
+<attribute name="NAME" x="308.61" y="342.9" size="1.778" layer="95" align="center-left"/>
+<attribute name="VALUE" x="308.61" y="340.36" size="1.778" layer="96" align="center-left"/>
+</instance>
 </instances>

Commit message: Add files via upload
Design process still on progress
Parts:
- added C6: 1uF/16v, rcl:C-EUC0603
- added R13: 10R, rcl:R-EU_R1206
- added R15: 2R2, rcl:R-EU_R2010
Connections:
- new net EXT_PWR_IN: IC3.VIN, IC6.INPUT, X2.2
- new net N$14: C6.2, IC2.AVCC, R13.2
- net GND: now also IC3.GND/ADJ, IC6.ADJ/GND, X2.1, X2.3
- net VCC: now also IC6.OUTPUT
Other:
- moved on the sheet: IC2, IC3, IC6
