File: PCB files/Metal Detector.sch (EAGLE design)
At the start: 122 parts, among them IC1 NE5534AD, IC2 BQ24133RGYR, IC3 LM317MBSTT3, IC4 ESP32-WROOM-32UE-N4, IC5 CP2102, IC6 LM317MBSTT3, J1 L-KLS1-TSJ3.5-013, J2 DG128-7.5, J2/BATTERY DG128-5.0-02P-14, Q1 IRF740, Q2 BC847AE6327HTSA1, Q3 SI2312CDS-T1-GE3, Q4 MBT3904DW1T1, Q5 SI2312CDS-T1-GE3, Q6 SI2323CDS-T1-GE3, Q7 BC847AE6327HTSA1, X2 DC21MMX

Commit message: Add files via upload
Redesigned Regulators Circuit and editing sheet
Parts:
- removed C10, C13: 1uF, resistor:CPOL-US085CS-1AR
- removed C11, C14: 10uF, resistor:CPOL-US085CS-1AR
- removed C39, C40: 0.1uF, rcl:C-EUC2012
- removed D10, D11, D6, D7: 1N4002, diode:1N4004
- removed FRAME3: FRAME-LEDGER, SparkFun-Aesthetics:FRAME-LEDGER
- removed IC3, IC6: LM317MBSTT3, v-reg:LM317MBSTT3
- removed J1: L-KLS1-TSJ3.5-013, L-KLS1-TSJ3.5-013:L-KLS1-TSJ3.5-013
- removed R14, R24: 240Ω, rcl:R-EU_R0805
- removed R16: 394Ω, rcl:R-EU_R0805
- removed R25: 720Ω, rcl:R-EU_R0805
- added C4, C5: 47uF, rcl:CPOL-EUSMCA
- added C41, C42: 10uF/25v, rcl:C-EUC1210
- added C43: (no value), rcl:CPOL-EUD
- added C44, C50: 0.047uF, rcl:C-EUC0603
- added C45: 4.7uF/10V, rcl:C-EUC0805
- added C46, C51: 47uF/6.3V, SparkFun-Capacitors:1.0UF-1206-50V-10%
- added C47, C48, C52, C53: 10uF/6.3V, rcl:C-EUC0805
- added C49, C54: 470pF, rcl:C-EUC0603
- added C55: 22nF, rcl:C-EUC0603
- added C57: 33nF, rcl:C-EUC0603
- added D14, D5: SS33-E3_57T, SS33-E3_57T:SS33-E3_57T
- added IC7: TPS54386PWPRG4, TPS54386PWPRG4:TPS54386PWPRG4
- added JP1: (no value), pinhead:PINHD-1X3
- added L2, L4: SRP7028AA-8R2M, SRP7028AA-8R2M:SRP7028AA-8R2M
- added R47, R6: 1KΩ, rcl:R-EU_R0603
- added R48, R49: 10Ω, rcl:R-EU_R0603
- added R50, R51: 20.5kΩ, rcl:R-EU_R0603
- added R52: 3.32kΩ, rcl:R-EU_R0603
- added R53: 6.49kΩ, rcl:R-EU_R0603
- added R55: 1.54kΩ, rcl:R-EU_R0603
- added R56: 3.83kΩ, rcl:R-EU_R0603
- R4: value 10kΩ -> 2.2kΩ
Connections:
- removed net ADC_PIN: IC1.OUT, R2.2
- removed net N$15: C11.+, D7.A, IC3.ADJ, R24.1, R25.2
- removed net N$20: C14.+, D11.A, IC6.ADJ, R14.1, R16.2
- removed net PULSE_PIN: R4.2
- new net FB1: C57.1, IC7.FB1, R51.2, R56.1
- new net FB2: C55.1, IC7.FB2, R50.2, R53.1
- new net N$32: C5.+, R47.1
- new net N$33: C4.-, JP1.1
- new net N$34: C5.-, JP1.2
- new net N$35: C44.2, IC7.BOOT2
- new net N$36: C44.1, C49.1, D5.K, IC7.SW2, L2.1
- new net N$37: C45.2, IC7.BP, IC7.ILIM2
- new net N$38: C55.2, R52.1
- new net N$39: C50.2, IC7.BOOT1
- new net N$40: C49.2, R48.1
- new net N$41: C57.2, R55.1
- new net N$42: C50.1, C54.1, D14.K, IC7.SW1, L4.1
- new net N$44: C54.2, R49.1
- new net N$8: C4.+, R6.1
- new net VCCIO: C46.1, C47.2, C48.2, DS1.A, L2.2, R11.1A, R17.2, R18.2, R50.1
- new net VCCIO1: C51.1, C52.2, C53.2, L4.2, R51.1
- net GND: now also C41.2, C42.2, C43.-, C45.1, C46.2, C47.1, C48.1, C51.2, C52.1, C53.1, D14.A, D5.A, IC7.!EN1, IC7.!EN2, IC7.EP, IC7.GND, JP1.3, R48.2, R49.2, R52.2, R53.2, R55.2, R56.2; no longer C10.-, C11.-, C13.-, C14.-, C39.2, C40.2, R16.1, R25.1
- net IO18: now also R4.2
- net IO25: now also R6.2
- net IO26: now also R47.2
- net IO4: now also IC1.OUT, R2.2
- net VCC: now also C41.1, C42.1, C43.+, IC7.PVDD1, IC7.PVDD2; no longer C10.+, C13.+, C39.1, C40.1, D10.A, D10.C, D11.C, D6.A, D6.C, D7.C, DS1.A, IC3.IN, IC3.OUT, IC6.IN, IC6.OUT, R11.1A, R14.2, R17.2, R18.2, R24.2
Other:
- note added: "5V & 3.3V BUCK CONVENTER"
- note added: "BATTERY CHARGE CIRCUIT"
- note added: "Buck Conventer Circuit"
- note added: "PI METAL DETECTOR CIRCUIT"
- note removed: "3.3V Voltage Regulator"
- note removed: "5V Voltage Regulator"
- note removed: "BATTERY CHARGE &POWER REGULATORS"
- moved on the sheet: C1, C12, C15, C16, C17, C18, C19, C2, C20, C21, C22, C23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

Commit message: Add files via upload
Redesigned Uaer Interface Block for Encoder (Encoder will include other design step)
Parts:
- removed R11, R12, R44: PC16S, piher:PC16S
- removed R46: 150Ω, rcl:R-EU_R0603
- added IC3: MCP4017T-503E_LT, MCP4017T-503E_LT:MCP4017T-503E_LT
- added Q8: BC847AE6327HTSA1, BC847AE6327HTSA1:BC847AE6327HTSA1
- added S1: (no value), switch:MS243
- C43: value (none) -> 100uF
Connections:
- removed net N$31: LS1.+, R12.1E
- new net N$15: DS1.VO, Q8.E
- new net N$20: IC3.B, LS1.+
- new net V_SYS_IN: C28.1, C35.1, Q6.S, R30.2, R31.2, S1.P
- net GND: now also C8.2, IC3.VSS; no longer R11.1E, R44.1E
- net IO18: no longer R4.2
- net IO19: now also R4.2
- net IO33: now also Q8.B
- net IO34: no longer R12.1S
- net IO35: no longer R11.1S
- net N$28: now also IC3.SCL; no longer DS1.VO, R44.1S
- net N$30: now also IC3.SDA; no longer C8.2, R12.1A, R46.2
- net PVCC: no longer C28.1, C35.1, Q6.S, R30.2, R31.2
- net VCC: now also IC3.VDD, IC3.W, Q8.C, S1.S; no longer R44.1A, R46.1
- net VCCIO: no longer R11.1A
Other:
- note added: "Power On-Off Button"
- note removed: "Sensitivity"
- moved on the sheet: C8, DS1, LS1, Q7, R45

Commit message: Add files via upload
Add connector to User Interface
Parts:
- removed DS1: WG12864B-TFH-V#N, NHD-12864WG-BTGH-T#N:NHD-12864WG-BTGH-T#N
- removed J2/BATTERY: DG128-5.0-02P-14, DG128-5.0-02P-14:DG128-5.0-02P-14
- removed JP1: (no value), pinhead:PINHD-1X3
- removed LS1: MCKPT-G1340-3917, MCKPT-G1340-3917:MCKPT-G1340-3917
- removed S1: (no value), switch:MS243
- removed U$1: 103AP-2, 130-AP2:103AP-2
- added J1: DG128-7.5, DG128-7.5-02P-14-00AH:DG128-7.5-02P-14-00AH
- added J3: DG129-5.0-03P-14-00AH, DG129-5.0-03P-14-00AH:DG129-5.0-03P-14-00AH
- added R11: 1kΩ, rcl:R-EU_R0603
- added R12: 560Ω, rcl:R-EU_R0603
- added X1: 22-23-2031, con-molex:22-23-2031
- added X3: 22-23-2051, con-molex:22-23-2051
- added X4: 22-23-2021, con-molex:22-23-2021
- added X5: 22-23-2091, con-molex:22-23-2091
Connections:
- removed net N$24: C31.1, C32.1, C33.1, J2/BATTERY.1, Q6.D, R33.2, R34.2
- removed net N$28: IC3.SCL
- removed net N$30: IC3.SDA
- removed net STAT: IC2.STAT
- new net N$31: Q8.B, R11.1
- net GND: now also J3.2, X1-3.S, X3-5.S, X5-2.S, X5-9.S; no longer DS1.K, DS1.VSS, J2/BATTERY.2, JP1.3, U$1.2
- net IO18: now also X5-7.S; no longer DS1.E
- net IO19: now also X5-4.S
- net IO21: now also IC3.SDA
- net IO22: now also IC3.SCL; no longer DS1.!RST
- net IO23: now also X5-5.S; no longer DS1.R/!W
- net IO33: now also R11.2; no longer Q8.B
- net IO34: now also X3-3.S
- net IO35: now also IC2.STAT
- net IO4: now also R12.1, R12.2
- net IO5: now also X5-6.S; no longer DS1.D/!I
- net N$15: now also X5-3.S; no longer DS1.VO
- net N$20: now also X4-1.S; no longer LS1.+
- net N$26: now also X4-2.S; no longer LS1.-
- net N$33: now also X1-1.S; no longer JP1.1
- net N$34: now also X1-2.S; no longer JP1.2
- net SENSOR_VN: now also X3-2.S
- net SENSOR_VP: now also X3-1.S
- net TS: now also J3.3; no longer U$1.1
- net VBATT: now also C31.1, C32.1, C33.1, J3.1, Q6.D, R33.2, R34.2
- net VCC: now also J1.1, X3-4.S, X5-1.S; no longer DS1.VDD, S1.S
- net VCCIO: now also X5-8.S; no longer DS1.A
- net V_SYS_IN: now also J1.2; no longer S1.P
Other:
- note added: "128 x 64 Graphic Display Circuit & Connector"
- note added: "Battery connector"
- note added: "Encoder connector"
- note added: "Headphone Connector"
- note added: "Speaker Circuit & Connector"
- note removed: "128 x 64 Graphic Display"
- note removed: "Headphone"
- note removed: "Speaker Buffer"
- moved on the sheet: Q7, Q8, R45

Commit message: Add files via upload
Separated USB to UART part edited User interface and Redesign Buck conventer Circuit for Implementation problem : /
Parts:
- removed C23: 100nF/ 50v, rcl:C-EUC0603
- removed C24: 4u7F/16v, rcl:C-EUC0603
- removed C41, C42: 10uF/25v, rcl:C-EUC1210
- removed C43: 100uF, rcl:CPOL-EUD
- removed C44, C50: 0.047uF, rcl:C-EUC0603
- removed C45: 4.7uF/10V, rcl:C-EUC0805
- removed C46, C51: 47uF/6.3V, SparkFun-Capacitors:1.0UF-1206-50V-10%
- removed C47, C48, C52, C53: 10uF/6.3V, rcl:C-EUC0805
- removed C49, C54: 470pF, rcl:C-EUC0603
- removed C55: 22nF, rcl:C-EUC0603
- removed C57: 33nF, rcl:C-EUC0603
- removed D14, D5: SS33-E3_57T, SS33-E3_57T:SS33-E3_57T
- removed IC7: TPS54386PWPRG4, TPS54386PWPRG4:TPS54386PWPRG4
- removed L2, L4: SRP7028AA-8R2M, SRP7028AA-8R2M:SRP7028AA-8R2M
- removed R48, R49: 10Ω, rcl:R-EU_R0603
- removed R50, R51: 20.5kΩ, rcl:R-EU_R0603
- removed R52: 3.32kΩ, rcl:R-EU_R0603
- removed R53: 6.49kΩ, rcl:R-EU_R0603
- removed R55: 1.54kΩ, rcl:R-EU_R0603
- removed R56: 3.83kΩ, rcl:R-EU_R0603
- added C10: 10uF/25V, rcl:C-EUC1210
- added C11: 3300pF, rcl:C-EUC0603
- added C13: 0.1uF, rcl:C-EUC0603
- added C14: 22uF/6.3V, rcl:C-EUC0805
- added IC6: TLV62130ARGTR, TLV62130ARGTR:TLV62130ARGTR
- added L3: IHLP2525CZER220M11, IHLP2525CZER220M11:IHLP2525CZER220M11
- added R14: 10KΩ, rcl:R-EU_R0603
- added R16: 0Ω, rcl:R-EU_R0603
- added R24: 100kΩ, rcl:R-EU_R0603
- added R25, R44: 680kΩ, rcl:R-EU_R1206
- added X7: (no value), con-molex:22-23-2061
- R19: value 4K7Ω -> 1KΩ
- R22: value 10KΩ -> 0Ω
Connections:
- removed net CLK: IC4.NC_4
- removed net CMD: IC4.NC_3
- removed net DCD: IC5.DCD
- removed net DSR: IC5.DSR
- removed net FB1: C57.1, IC7.FB1, R51.2, R56.1
- removed net FB2: C55.1, IC7.FB2, R50.2, R53.1
- removed net N$35: C44.2, IC7.BOOT2
- removed net N$36: C44.1, C49.1, D5.K, IC7.SW2, L2.1
- removed net N$37: C45.2, IC7.BP, IC7.ILIM2
- removed net N$38: C55.2, R52.1
- removed net N$39: C50.2, IC7.BOOT1
- removed net N$40: C49.2, R48.1
- removed net N$41: C57.2, R55.1
- removed net N$42: C50.1, C54.1, D14.K, IC7.SW1, L4.1
- removed net N$44: C54.2, R49.1
- removed net REGIN: C23.2, C24.2, IC5.REGIN
- removed net RI: IC5.RI
- removed net SD0: IC4.NC_5
- removed net SD1: IC4.NC_6
- removed net SD2: IC4.NC_1
- removed net SD3: IC4.NC_2
- removed net VBUS_CP: C25.2, C26.2, IC5.VBUS
- removed net VCCIO1: C51.1, C52.2, C53.2, L4.2, R51.1
- removed net V_SYS_IN: C28.1, C35.1, J1.2, Q6.S, R30.2, R31.2
- new net N$24: IC5.!RST, R19.1
- new net N$28: IC6.PG, R24.1
- new net N$30: IC6.FB, R25.2, R44.1
- new net N$49: IC6.SW_1, IC6.SW_2, IC6.SW_3, L3.1
- new net RXD: IC5.RXD, R16.2, X7-1.S
- new net TXD: IC5.TXD, R22.2, X7-2.S
- new net VCCINT: J1.2
- net 3V3: now also R18.2, X7-5.S
- net ACTıVE: now also R14.1
- net EN: now also S3.1, X7-3.S; no longer S3.2
- net GND: now also C10.2, C11.2, C13.2, C14.1, IC6.AGND, IC6.DEF, IC6.EXPOSED_THERMAL_PAD, IC6.FSW, IC6.PGND_1, IC6.PGND_2, R14.2, R44.2, S3.2, S4.2, X7-6.S; no longer C23.1, C24.1, C41.2, C42.2, C43.-, C45.1, C46.2, C47.1, C48.1, C51.2, C52.1, C53.1, D14.A, D5.A, IC7.!EN1, IC7.!EN2, IC7.EP, IC7.GND, R19.1, R48.2, R49.2, R52.2, R53.2, R55.2, R56.2, S3.1, S4.1
- net IO0: now also S4.1, X7-4.S; no longer S4.2
- net IO13: no longer IC5.RTS
- net IO15: no longer IC5.CTS
- net IO2: no longer R19.2
- net IO23: no longer IC4.NC_7
- net N$19: now also C11.1, IC6.SS/TR; no longer IC5.TXD, R22.1
- net PVCC: now also C28.1, C35.1, Q6.S, R30.2, R31.2
- net RTS: now also IC5.RTS
- net RXD0: now also R22.1; no longer R22.2
- net TXD0: now also R16.1; no longer IC5.RXD
- net VCC: now also C10.1, C13.1, C14.2, C25.2, C26.2, IC5.VBUS, IC6.AVIN, IC6.EN, IC6.PVIN_1, IC6.PVIN_2, IC6.VOS, L3.2, R24.2, R25.1; no longer C41.1, C42.1, C43.+, IC7.PVDD1, IC7.PVDD2
- net VCCIO: no longer C46.1, C47.2, C48.2, L2.2, R18.2, R50.1
- net VDD_CP: now also IC5.REGIN, R19.2
Other:
- note added: "5V Buck Conventer Circuit"
- note added: "Serial Signal Connection"
- note removed: "Buck Conventer Circuit"
- note removed: "De-Coupling Capacitors"
- moved on the sheet: C17, C18, C19, C20, C21, C22, C25, C26, D4, D8, D9, F2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

Commit message: Add files via upload
Designed buck conventer and linear voltage regulator circuit and simulated circuit on TI platform next progress change opamp for offset voltage implementation issue and redesign headphone connection after that All design will on last checking process before drawing layout
Parts:
- added C23, C24: 10uF/16V, rcl:CPOL-EUB
- added D5: ES1B-E3_61T, ES1B-E3_61T:ES1B-E3_61T
- added IC7: TLV1117-33IDCYR, TLV1117-33IDCYR:TLV1117-33IDCYR
- R44: value 680kΩ -> 130kΩ
Connections:
- removed net 3V3: C19.2, C20.2, IC4.3V3, R18.2, X7-5.S
- removed net PVCC: C28.1, C35.1, IC2.PVCC_1, IC2.PVCC_2, Q6.S, R30.2, R31.2
- removed net VDD_CP: C21.2, C22.2, IC5.REGIN, IC5.VDD, R19.2
- net GND: now also C23.-, C24.-, IC7.ADJ/GND
- net VCC: now also C23.+, D5.K, IC7.INPUT
- net VCCINT: now also C28.1, C35.1, IC2.PVCC_1, IC2.PVCC_2, Q6.S, R30.2, R31.2
- net VCCIO: now also C19.2, C20.2, C21.2, C22.2, C24.+, D5.A, IC4.3V3, IC5.REGIN, IC5.VDD, IC7.OUTPUT_1, IC7.OUTPUT_2, R18.2, R19.2, X7-5.S
Other:
- note added: "3.3V Linear Voltage Regulator"
