File: PCB files/Metal Detector.sch (EAGLE design)
At the start: 110 parts, among them IC1 NE5534AD, IC2 BQ24133RGYR, IC3 TPS54228DDAR, IC4 ESP32-WROOM-32UE-N4, IC7 TLV1117-33IDCYR, J2 DG128-7.5, Q1 IRF740, Q11 MMBT3904, Q2 IRF740, Q3 IRF9630, Q4 IRF740, Q9 MMBT3904, X2 DC21MMX

Commit message: Add files via upload
Designed 5V, 3.3V power circuit and signal processing circuit after that repositioned component I will do microprossesor connection and repositioning on next section
Parts:
- removed L2: SRP1265A-4R7M, SRP1265A-4R7M:SRP1265A-4R7M
- removed TR2: 100K, rcl:R-TRIMM3296X
- added L3: SRU8043-4R7Y, SRU8043-330Y:SRU8043-330Y
- added R8: 3224W-1-104E, 3224W-1-104E:3224W-1-104E
Connections:
- net N$10: now also R8.WIPER; no longer TR2.S
- net N$11: now also R8.CW; no longer TR2.E
- net N$19: now also L3.1; no longer L2.1
- net N$9: now also R8.CCW; no longer TR2.A
- net VCC: now also L3.2; no longer L2.2
Other:
- moved on the sheet: C7, R10
Changed lines of the file:
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@@
 <part name="D2" library="diode" library_urn="urn:adsk.eagle:library:210" deviceset="1N4148" device="DO35-7" package3d_urn="urn:adsk.eagle:package:43339/2"/>
 <part name="D3" library="diode" library_urn="urn:adsk.eagle:library:210" deviceset="1N4148" device="DO35-7" package3d_urn="urn:adsk.eagle:package:43339/2"/>
-<part name="TR2" library="rcl" library_urn="urn:adsk.eagle:library:334" deviceset="R-TRIMM" device="3296X" package3d_urn="urn:adsk.eagle:package:26034/1" value="100K"/>
 <part name="C7" library="SparkFun-Capacitors" library_urn="urn:adsk.eagle:library:510" deviceset="10UF" device="-0402T-6.3V-20%" package3d_urn="urn:adsk.eagle:package:41385069/1" value="10uF"/>
 <part name="IC4" library="ESP32-WROOM-32UE-N4" deviceset="ESP32-WROOM-32UE-N4" device=""/>
@@
 <part name="GND18" library="SparkFun-Aesthetics" deviceset="GND" device=""/>
 <part name="GND19" library="SparkFun-Aesthetics" deviceset="GND" device=""/>
-<part name="L2" library="SRP1265A-4R7M" deviceset="SRP1265A-4R7M" device=""/>
 <part name="SUPPLY2" library="supply2" library_urn="urn:adsk.eagle:library:372" deviceset="VCC" device="" value="SYS_VCC"/>
+<part name="L3" library="SRU8043-330Y" deviceset="SRU8043-330Y" device="" value="SRU8043-4R7Y"/>
+<part name="R8" library="3224W-1-104E" deviceset="3224W-1-104E" device=""/>
 </parts>
 <sheets>
@@
 <attribute name="VALUE" x="456.9714" y="345.44" size="1.778" layer="96" rot="R90"/>
 </instance>
-<instance part="TR2" gate="G$1" x="487.68" y="365.76" smashed="yes" rot="MR180">
-<attribute name="NAME" x="488.95" y="369.951" size="1.778" layer="95" rot="MR180"/>
-<attribute name="VALUE" x="488.95" y="364.49" size="1.778" layer="96" rot="MR180"/>
-</instance>
-<instance part="C7" gate="G$1" x="508" y="379.73" smashed="yes" rot="R180">
-<attribute name="NAME" x="514.096" y="376.809" size="1.778" layer="95" font="vector" rot="R180"/>
-<attribute name="VALUE" x="514.096" y="381.889" size="1.778" layer="96" font="vector" rot="R180"/>
+<instance part="C7" gate="G$1" x="533.4" y="379.73" smashed="yes" rot="R180">
+<attribute name="NAME" x="539.496" y="376.809" size="1.778" layer="95" font="vector" rot="R180"/>
+<attribute name="VALUE" x="539.496" y="381.889" size="1.778" layer="96" font="vector" rot="R180"/>
 </instance>
 <instance part="IC4" gate="G$1" x="378.46" y="508" smashed="yes">
@@
 <attribute name="VALUE" x="467.36" y="340.36" size="1.778" layer="96"/>
 </instance>
-<instance part="GND34" gate="1" x="508" y="370.84" smashed="yes">
-<attribute name="VALUE" x="505.46" y="368.3" size="1.778" layer="96"/>
+<instance part="GND34" gate="1" x="533.4" y="370.84" smashed="yes">
+<attribute name="VALUE" x="530.86" y="368.3" size="1.778" layer="96"/>
 </instance>
 <instance part="GND35" gate="1" x="477.52" y="370.84" smashed="yes">
@@
 <attribute name="VALUE" x="434.34" y="294.64" size="1.778" layer="96"/>
 </instance>
-<instance part="P+1" gate="VCC" x="500.38" y="391.16" smashed="yes">
-<attribute name="VALUE" x="500.38" y="391.16" size="1.778" layer="96"/>
+<instance part="P+1" gate="VCC" x="525.78" y="391.16" smashed="yes">
+<attribute name="VALUE" x="525.78" y="391.16" size="1.778" layer="96"/>
 </instance>
 <instance part="C12" gate="G$1" x="477.52" y="379.984" smashed="yes">
@@
 <attribute name="VALUE" x="482.6" y="342.265" size="1.778" layer="96"/>
 </instance>
-<instance part="R10" gate="G$1" x="500.38" y="373.38" smashed="yes" rot="R90">
-<attribute name="NAME" x="498.8814" y="369.57" size="1.778" layer="95" rot="R90"/>
-<attribute name="VALUE" x="503.682" y="369.57" size="1.778" layer="96" rot="R90"/>
+<instance part="R10" gate="G$1" x="525.78" y="373.38" smashed="yes" rot="R90">
+<attribute name="NAME" x="524.2814" y="369.57" size="1.778" layer="95" rot="R90"/>
+<attribute name="VALUE" x="529.082" y="369.57" size="1.778" layer="96" rot="R90"/>
 </instance>
 <instance part="GND32" gate="1" x="492.76" y="320.04" smashed="yes">
@@
 <attribute name="VALUE" x="180.34" y="231.14" size="1.778" layer="96"/>
 </instance>
-<instance part="L2" gate="G$1" x="149.86" y="266.7" smashed="yes">
-<attribute name="NAME" x="151.13" y="273.05" size="1.778" layer="95" align="center-left"/>
-<attribute name="VALUE" x="151.13" y="270.51" size="1.778" layer="96" align="center-left"/>
-</instance>
 <instance part="SUPPLY2" gate="G$1" x="248.92" y="525.78" smashed="yes">
 <attribute name="VALUE" x="247.015" y="528.955" size="1.778" layer="96"/>
+</instance>
+<instance part="L3" gate="G$1" x="149.86" y="266.7" smashed="yes">
+<attribute name="NAME" x="166.37" y="273.05" size="1.778" layer="95" align="center-left"/>
+<attribute name="VALUE" x="166.37" y="270.51" size="1.778" layer="96" align="center-left"/>
+</instance>
+<instance part="R8" gate="G$1" x="518.16" y="365.76" smashed="yes" rot="R180">
+<attribute name="NAME" x="511.81" y="375.92" size="1.778" layer="95" rot="R180" align="center-left"/>
+<attribute name="VALUE" x="511.81" y="373.38" size="1.778" layer="96" rot="R180" align="center-left"/>
 </instance>
 </instances>
@@
 <pinref part="C7" gate="G$1" pin="1"/>
 <pinref part="GND34" gate="1" pin="GND"/>
-<wire x1="508" y1="374.65" x2="508" y2="373.38" width="0.1524" layer="91"/>
+<wire x1="533.4" y1="374.65" x2="533.4" y2="373.38" width="0.1524" layer="91"/>
 </segment>
 <segment>
@@
 <segment>
 <pinref part="P+1" gate="VCC" pin="VCC"/>
-<wire x1="500.38" y1="388.62" x2="500.38" y2="383.54" width="0.1524" layer="91"/>
+<wire x1="525.78" y1="388.62" x2="525.78" y2="383.54" width="0.1524" layer="91"/>
 <pinref part="R10" gate="G$1" pin="2"/>
 <pinref part="C7" gate="G$1" pin="2"/>
-<wire x1="500.38" y1="383.54" x2="500.38" y2="378.46" width="0.1524" layer="91"/>
-<wire x1="508" y1="382.27" x2="508" y2="383.54" width="0.1524" layer="91"/>
-<wire x1="508" y1="383.54" x2="500.38" y2="383.54" width="0.1524" layer="91"/>
-<junction x="500.38" y="383.54"/>
+<wire x1="525.78" y1="383.54" x2="525.78" y2="378.46" width="0.1524" layer="91"/>
+<wire x1="533.4" y1="382.27" x2="533.4" y2="383.54" width="0.1524" layer="91"/>
+<wire x1="533.4" y1="383.54" x2="525.78" y2="383.54" width="0.1524" layer="91"/>
+<junction x="525.78" y="383.54"/>
 </segment>
 <segment>
@@
 <wire x1="177.8" y1="266.7" x2="182.88" y2="266.7" width="0.1524" layer="91"/>
 <wire x1="182.88" y1="266.7" x2="182.88" y2="264.16" width="0.1524" layer="91"/>
-<pinref part="L2" gate="G$1" pin="2"/>
 <wire x1="170.18" y1="266.7" x2="172.72" y2="266.7" width="0.1524" layer="91"/>
 <junction x="172.72" y="266.7"/>
@@
 <wire x1="177.8" y1="226.06" x2="177.8" y2="266.7" width="0.1524" layer="91"/>
 <junction x="177.8" y="266.7"/>
+<pinref part="L3" gate="G$1" pin="2"/>
 </segment>
 <segment>
@@
 <wire x1="482.6" y1="365.76" x2="482.6" y2="373.38" width="0.1524" layer="91"/>
 <wire x1="482.6" y1="373.38" x2="487.68" y2="373.38" width="0.1524" layer="91"/>
-<pinref part="TR2" gate="G$1" pin="A"/>
-<wire x1="487.68" y1="373.38" x2="487.68" y2="370.84" width="0.1524" layer="91"/>
 <pinref part="IC1" gate="A" pin="ON"/>
 <wire x1="472.44" y1="363.22" x2="472.44" y2="365.76" width="0.1524" layer="91"/>
 <wire x1="472.44" y1="365.76" x2="482.6" y2="365.76" width="0.1524" layer="91"/>
+<wire x1="487.68" y1="373.38" x2="487.68" y2="368.3" width="0.1524" layer="91"/>
+<pinref part="R8" gate="G$1" pin="CCW"/>
+<wire x1="487.68" y1="368.3" x2="490.22" y2="368.3" width="0.1524" layer="91"/>
 </segment>
 </net>
 <net name="N$11" class="0">
 <segment>
-<pinref part="TR2" gate="G$1" pin="E"/>
-<wire x1="487.68" y1="360.68" x2="487.68" y2="358.14" width="0.1524" layer="91"/>
 <pinref part="IC1" gate="A" pin="ON/CMP"/>
 <wire x1="487.68" y1="358.14" x2="480.06" y2="358.14" width="0.1524" layer="91"/>
@@
 <pinref part="C2" gate="G$1" pin="2"/>
 <wire x1="483.616" y1="345.44" x2="487.68" y2="345.44" width="0.1524" layer="91"/>
+<wire x1="487.68" y1="358.14" x2="487.68" y2="365.76" width="0.1524" layer="91"/>
+<pinref part="R8" gate="G$1" pin="CW"/>
+<wire x1="487.68" y1="365.76" x2="490.22" y2="365.76" width="0.1524" layer="91"/>
 </segment>
 </net>
 <net name="N$10" class="0">
 <segment>
-<pinref part="TR2" gate="G$1" pin="S"/>
-<wire x1="492.76" y1="365.76" x2="500.38" y2="365.76" width="0.1524" layer="91"/>
-<wire x1="500.38" y1="365.76" x2="500.38" y2="368.3" width="0.1524" layer="91"/>
+<wire x1="518.16" y1="365.76" x2="525.78" y2="365.76" width="0.1524" layer="91"/>
+<wire x1="525.78" y1="365.76" x2="525.78" y2="368.3" width="0.1524" layer="91"/>
 <pinref part="R10" gate="G$1" pin="1"/>
+<pinref part="R8" gate="G$1" pin="WIPER"/>
 </segment>
 </net>
@@
 <pinref part="IC3" gate="G$1" pin="SW"/>
 <wire x1="134.62" y1="266.7" x2="144.78" y2="266.7" width="0.1524" layer="91"/>
-<wire x1="144.78" y1="266.7" x2="149.86" y2="266.7" width="0.1524" layer="91"/>
+<pinref part="L3" gate="G$1" pin="1"/>
+<wire x1="149.86" y1="266.7" x2="144.78" y2="266.7" width="0.1524" layer="91"/>
 <junction x="144.78" y="266.7"/>
-<pinref part="L2" gate="G$1" pin="1"/>
-</segment>
-</net>
+</segment>
+</net>

Commit message: Add files via upload
All schematic and board design process is done after that upload BOM file, 3rd view docs and manufacturing files
Parts:
- removed C7: 10uF, SparkFun-Capacitors:10UF-0402T-6.3V-20%
- added C39: 10uF, rcl:C-EUC0603
- R2: value 1mΩ -> 0.01Ω
- R30, R31: value 10KΩ -> 10kΩ
Connections:
- net GND: now also C39.2; no longer C7.1
- net VCC: now also C39.1; no longer C7.2
Changed lines of the file:
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@@
 <part name="D2" library="diode" library_urn="urn:adsk.eagle:library:210" deviceset="1N4148" device="DO35-7" package3d_urn="urn:adsk.eagle:package:43339/2"/>
 <part name="D3" library="diode" library_urn="urn:adsk.eagle:library:210" deviceset="1N4148" device="DO35-7" package3d_urn="urn:adsk.eagle:package:43339/2"/>
-<part name="C7" library="SparkFun-Capacitors" library_urn="urn:adsk.eagle:library:510" deviceset="10UF" device="-0402T-6.3V-20%" package3d_urn="urn:adsk.eagle:package:41385069/1" value="10uF"/>
 <part name="IC4" library="ESP32-WROOM-32UE-N4" deviceset="ESP32-WROOM-32UE-N4" device=""/>
 <part name="GND8" library="supply1" library_urn="urn:adsk.eagle:library:371" deviceset="GND" device=""/>
@@
 <part name="SUPPLY1" library="supply2" library_urn="urn:adsk.eagle:library:372" deviceset="VCC" device="" value="SYS_VCC"/>
 <part name="R7" library="rcl" library_urn="urn:adsk.eagle:library:334" deviceset="R-EU_" device="0207/10" package3d_urn="urn:adsk.eagle:package:23491/2" value="1Ω"/>
-<part name="R2" library="rcl" library_urn="urn:adsk.eagle:library:334" deviceset="R-EU_" device="R1206" package3d_urn="urn:adsk.eagle:package:23540/2" value="1mΩ"/>
+<part name="R2" library="rcl" library_urn="urn:adsk.eagle:library:334" deviceset="R-EU_" device="R1206" package3d_urn="urn:adsk.eagle:package:23540/2" value="0.01Ω"/>
 <part name="R9" library="rcl" library_urn="urn:adsk.eagle:library:334" deviceset="R-EU_" device="R1206" package3d_urn="urn:adsk.eagle:package:23540/2" value="1kΩ"/>
 <part name="C1" library="rcl" library_urn="urn:adsk.eagle:library:334" deviceset="C-EU" device="C0603" package3d_urn="urn:adsk.eagle:package:23616/2" value="15pF"/>
@@
 <part name="R20" library="WSL1206R0100FEK18" deviceset="WSL1206R0100FEK18" device=""/>
 <part name="R19" library="rcl" library_urn="urn:adsk.eagle:library:334" deviceset="R-EU_" device="R1206" package3d_urn="urn:adsk.eagle:package:23540/2" value="20Ω"/>
-<part name="R30" library="rcl" library_urn="urn:adsk.eagle:library:334" deviceset="R-EU_" device="R1206" package3d_urn="urn:adsk.eagle:package:23540/2" value="10KΩ"/>
-<part name="R31" library="rcl" library_urn="urn:adsk.eagle:library:334" deviceset="R-EU_" device="R1206" package3d_urn="urn:adsk.eagle:package:23540/2" value="10KΩ"/>
+<part name="R30" library="rcl" library_urn="urn:adsk.eagle:library:334" deviceset="R-EU_" device="R1206" package3d_urn="urn:adsk.eagle:package:23540/2" value="10kΩ"/>
+<part name="R31" library="rcl" library_urn="urn:adsk.eagle:library:334" deviceset="R-EU_" device="R1206" package3d_urn="urn:adsk.eagle:package:23540/2" value="10kΩ"/>
 <part name="R33" library="rcl" library_urn="urn:adsk.eagle:library:334" deviceset="R-EU_" device="R1206" package3d_urn="urn:adsk.eagle:package:23540/2" value="2.2kΩ"/>
 <part name="R1" library="WSL1206R0100FEK18" deviceset="WSL1206R0100FEK18" device="" value="WSL1206R0200FEK18"/>
@@
 <part name="L3" library="SRU8043-330Y" deviceset="SRU8043-330Y" device="" value="SRU8043-4R7Y"/>
 <part name="R8" library="3224W-1-104E" deviceset="3224W-1-104E" device=""/>
+<part name="C39" library="rcl" library_urn="urn:adsk.eagle:library:334" deviceset="C-EU" device="C0603" package3d_urn="urn:adsk.eagle:package:23616/2" value="10uF"/>
 </parts>
 <sheets>
@@
 <attribute name="VALUE" x="456.9714" y="345.44" size="1.778" layer="96" rot="R90"/>
 </instance>
-<instance part="C7" gate="G$1" x="533.4" y="379.73" smashed="yes" rot="R180">
-<attribute name="NAME" x="539.496" y="376.809" size="1.778" layer="95" font="vector" rot="R180"/>
-<attribute name="VALUE" x="539.496" y="381.889" size="1.778" layer="96" font="vector" rot="R180"/>
-</instance>
 <instance part="IC4" gate="G$1" x="378.46" y="508" smashed="yes">
 <attribute name="NAME" x="407.67" y="513.08" size="1.778" layer="95" align="center-left"/>
@@
 <attribute name="NAME" x="511.81" y="375.92" size="1.778" layer="95" rot="R180" align="center-left"/>
 <attribute name="VALUE" x="511.81" y="373.38" size="1.778" layer="96" rot="R180" align="center-left"/>
+</instance>
+<instance part="C39" gate="G$1" x="533.4" y="379.984" smashed="yes">
+<attribute name="NAME" x="534.924" y="380.365" size="1.778" layer="95"/>
+<attribute name="VALUE" x="533.4" y="375.285" size="1.778" layer="96"/>
 </instance>
 </instances>
@@
 </segment>
 <segment>
-<pinref part="C7" gate="G$1" pin="1"/>
-<pinref part="GND34" gate="1" pin="GND"/>
-<wire x1="533.4" y1="374.65" x2="533.4" y2="373.38" width="0.1524" layer="91"/>
-</segment>
-<segment>
 <pinref part="Q1" gate="G$1" pin="S"/>
 <pinref part="GND11" gate="1" pin="GND"/>
@@
 <wire x1="182.88" y1="256.54" x2="182.88" y2="236.22" width="0.1524" layer="91"/>
 </segment>
+<segment>
+<pinref part="C39" gate="G$1" pin="2"/>
+<pinref part="GND34" gate="1" pin="GND"/>
+<wire x1="533.4" y1="374.904" x2="533.4" y2="373.38" width="0.1524" layer="91"/>
+</segment>
 </net>
 <net name="VCC" class="0">
@@
 <wire x1="525.78" y1="388.62" x2="525.78" y2="383.54" width="0.1524" layer="91"/>
 <pinref part="R10" gate="G$1" pin="2"/>
-<pinref part="C7" gate="G$1" pin="2"/>
 <wire x1="525.78" y1="383.54" x2="525.78" y2="378.46" width="0.1524" layer="91"/>
-<wire x1="533.4" y1="382.27" x2="533.4" y2="383.54" width="0.1524" layer="91"/>
+<wire x1="533.4" y1="382.524" x2="533.4" y2="383.54" width="0.1524" layer="91"/>
 <wire x1="533.4" y1="383.54" x2="525.78" y2="383.54" width="0.1524" layer="91"/>
 <junction x="525.78" y="383.54"/>
-</segment>
-<segment>
+<pinref part="C39" gate="G$1" pin="1"/>
+</segment>
+<segment>

Commit message: Add files via upload
Edited pcb trace nad add test point
Parts:
- removed C4, C5: 47uF, rcl:CPOL-EUSMCA
- added TP1, TP2, TP3, TP4, TP5, TP6, TP7, TP8: TPTP10R, testpad:TPTP10R
- C19: value 100uF/ 6.3V -> 100uF/6.3V; device rcl:C-EUC0603 -> rcl:C-EUC1206
- DISPLAY: value (none) -> L-KLS1-2.50-09-S
- ENCODER: value (none) -> L-KLS1-2.50-05-S
- HEADPHONE: value (none) -> L-KLS1-XL4-2.50-04-R
- ON-OFF, SPEAKER: value (none) -> L-KLS1-XL4-2.50-02-R
- SERIAL: value (none) -> L-KLS1-2.50-06-S
- renumbered X2 to 12VIN
Connections:
- removed net N$20: C5.-, HEADPHONE-3.S
- removed net N$26: C4.-, HEADPHONE-2.S
- net 12V_IN: now also TP6.TP
- net IO0: now also TP1.TP
- net IO4: now also TP8.TP
- net N$32: now also HEADPHONE-3.S; no longer C5.+
- net N$8: now also HEADPHONE-2.S; no longer C4.+
- net VBATT: now also TP4.TP
- net VCC: now also TP2.TP, TP5.TP
- net VCCIO: now also TP3.TP, TP7.TP
