File: PCB files/Metal Detector.brd (EAGLE design)
At the start: 100 x 80 mm, 139 parts, among them IC1 NE5534AD, IC2 BQ24133RGYR, IC3 MCP4017T-503E_LT, IC4 ESP32-WROOM-32UE-N4, IC5 CP2102, IC7 TPS54386PWPRG4, J1 DG128-7.5, J2 DG128-7.5, J3 DG129-5.0-03P-14-00AH, Q1 IRF740, Q2 BC847AE6327HTSA1, Q3 SI2312CDS-T1-GE3, Q4 MBT3904DW1T1, Q5 SI2312CDS-T1-GE3, Q6 SI2323CDS-T1-GE3, Q7 BC847AE6327HTSA1, Q8 BC847AE6327HTSA1, X1 22-23-2031, X2 DC21MMX, X3 22-23-2051, X4 22-23-2021, X5 22-23-2091

Commit message: Add files via upload
Separated USB to UART part edited User interface and Redesign Buck conventer Circuit for Implementation problem : /
Parts:
- removed C23: 100nF/ 50v, rcl:C0603
- removed C24: 4u7F/16v, rcl:C0603
- removed C41, C42: 10uF/25v, rcl:C1210
- removed C43: 100uF, rcl:PANASONIC_D
- removed C44, C50: 0.047uF, rcl:C0603
- removed C45: 4.7uF/10V, rcl:C0805
- removed C46, C51: 47uF/6.3V, SparkFun-Capacitors:1206
- removed C47, C48, C52, C53: 10uF/6.3V, rcl:C0805
- removed C49, C54: 470pF, rcl:C0603
- removed C55: 22nF, rcl:C0603
- removed C57: 33nF, rcl:C0603
- removed D14, D5: SS33-E3_57T, SS33-E3_57T:DIOM7959X262N
- removed IC7: TPS54386PWPRG4, TPS54386PWPRG4:SOP65P640X120-15N
- removed L2, L4: SRP7028AA-8R2M, SRP7028AA-8R2M:INDPM7166X300N
- removed R48, R49: 10Ω, rcl:R0603
- removed R50, R51: 20.5kΩ, rcl:R0603
- removed R52: 3.32kΩ, rcl:R0603
- removed R53: 6.49kΩ, rcl:R0603
- removed R55: 1.54kΩ, rcl:R0603
- removed R56: 3.83kΩ, rcl:R0603
- added C10: 10uF/25V, rcl:C1210
- added C11: 3300pF, rcl:C0603
- added C13: 0.1uF, rcl:C0603
- added C14: 22uF/6.3V, rcl:C0805
- added IC6: TLV62130ARGTR, TLV62130ARGTR:QFN50P300X300X100-17N
- added L3: IHLP2525CZER220M11, IHLP2525CZER220M11:INDPM6965X300N
- added R14: 10KΩ, rcl:R0603
- added R16: 0Ω, rcl:R0603
- added R24: 100kΩ, rcl:R0603
- added R25, R44: 680kΩ, rcl:R1206
- added X7: (no value), con-molex:22-23-2061
- R19: value 4K7Ω -> 1KΩ
- R22: value 10KΩ -> 0Ω
- moved R19 1106.1 mm to (-221.0, -1144.3)
- moved R22 1103.4 mm to (-221.0, -1139.2)
Connections:
- removed net CLK: IC4.20
- removed net CMD: IC4.19
- removed net DCD: IC5.1
- removed net DSR: IC5.27
- removed net FB1: C57.1, IC7.7, R51.2, R56.1
- removed net FB2: C55.1, IC7.8, R50.2, R53.1
- removed net N$35: C44.2, IC7.13
- removed net N$36: C44.1, C49.1, D5.1, IC7.12, L2.1
- removed net N$37: C45.2, IC7.11, IC7.9
- removed net N$38: C55.2, R52.1
- removed net N$39: C50.2, IC7.2
- removed net N$40: C49.2, R48.1
- removed net N$41: C57.2, R55.1
- removed net N$42: C50.1, C54.1, D14.1, IC7.3, L4.1
- removed net N$44: C54.2, R49.1
- removed net REGIN: C23.2, C24.2, IC5.7
- removed net RI: IC5.2
- removed net SD0: IC4.21
- removed net SD1: IC4.22
- removed net SD2: IC4.17
- removed net SD3: IC4.18
- removed net VBUS_CP: C25.2, C26.2, IC5.8
- removed net VCCIO1: C51.1, C52.2, C53.2, L4.2, R51.1
- removed net V_SYS_IN: C28.1, C35.1, J1.2, Q6.2, R30.2, R31.2
- new net N$24: IC5.9, R19.1
- new net N$28: IC6.4, R24.1
- new net N$30: IC6.5, R25.2, R44.1
- new net N$49: IC6.1, IC6.2, IC6.3, L3.1
- new net RXD: IC5.25, R16.2, X7.1
- new net TXD: IC5.26, R22.2, X7.2
- new net VCCINT: J1.2
- net 3V3: now also R18.2, X7.5
- net ACTıVE: now also R14.1
- net EN: now also S3.1, S3.2, X7.3; no longer S3.3, S3.4
- net GND: now also C10.2, C11.2, C13.2, C14.1, IC6.15, IC6.16, IC6.17, IC6.6, IC6.7, IC6.8, R14.2, R44.2, S3.3, S3.4, S4.3, S4.4, X7.6; no longer C23.1, C24.1, C41.2, C42.2, C43.-, C45.1, C46.2, C47.1, C48.1, C51.2, C52.1, C53.1, D14.2, D5.2, IC7.15, IC7.4, IC7.5, IC7.6, R19.1, R48.2, R49.2, R52.2, R53.2, R55.2, R56.2, S3.1, S3.2, S4.1, S4.2
- net IO0: now also S4.1, S4.2, X7.4; no longer S4.3, S4.4
- net IO13: no longer IC5.24
- net IO15: no longer IC5.23
- net IO2: no longer R19.2
- net IO23: no longer IC4.32
- net N$19: now also C11.1, IC6.9; no longer IC5.26, R22.1
- net PVCC: now also C28.1, C35.1, Q6.2, R30.2, R31.2
- net RTS: now also IC5.24
- net RXD0: now also R22.1; no longer R22.2
- net TXD0: now also R16.1; no longer IC5.25
- net VCC: now also C10.1, C13.1, C14.2, C25.2, C26.2, IC5.8, IC6.10, IC6.11, IC6.12, IC6.13, IC6.14, L3.2, R24.2, R25.1; no longer C41.1, C42.1, C43.+, IC7.1, IC7.14
- net VCCIO: no longer C46.1, C47.2, C48.2, L2.2, R18.2, R50.1
- net VDD_CP: now also IC5.7, R19.2
